File: kicad controllers/deltavr_controller/deltavr_controller.kicad_sch (KiCad schematic)
At the start: 52 parts, among them J1 debug, J2 battery pins 3.7v, J3 test 3.3v pins, Q1 IRLZ44N, SW1 SW_Push, SW2 SW_Push, SW3 SW_Push, U10 ADS1115IDGS, U2 nice_nano, U3 SS49E, U4 SS49E, U5 LSM6DSVTR, U6 HT7333, U7 HT7333, U8 HT7333, U9 HT7333

Commit message: controllers are FUVCKING DONNE AYYYAYYYY
Parts:
- removed D5, D6, D7, D8: 850nm, LED_THT:LED_D5.0mm_IRGrey, symbol LED:SFH4550
- removed R10, R11, R12, R13: 15Ω, Resistor_SMD:R_0603_1608Metric_Pad0.98x0.95mm_HandSolder, symbol Device:R
- removed U6, U7: HT7333, Package_TO_SOT_SMD:SOT-89-3, symbol Regulator_Linear:HT75xx-1-SOT89
- added C18: 10uF, Capacitor_SMD:C_0603_1608Metric_Pad1.08x0.95mm_HandSolder, symbol Device:C
- added C19: 100nF, Capacitor_SMD:C_0603_1608Metric_Pad1.08x0.95mm_HandSolder, symbol Device:C
- added R1, R2: 4.7kΩ, Resistor_SMD:R_0603_1608Metric_Pad0.98x0.95mm_HandSolder, symbol Device:R
- added U1: NRF24L01_Breakout, RF_Module:nRF24L01_Breakout, symbol RF:NRF24L01_Breakout
- U3, U4: footprint SEN3_SS49E_HNW -> ss49e footprint:SEN3_SS49E_HNW
Connections:
- net 1 - SDO/SAO: now also U1.7 (MISO)
- net 13 - SCL: now also U1.5 (SCK)
- net 14 - SDA: now also U1.6 (MOSI)
- net 2 - SDX: now also C2.2, C3.1, C4.2, C5.2, C18.2, C19.2, U1.1 (GND)
- net 3.3v: now also C18.1, C19.1, R1.2, R2.2, U1.2 (VCC); no longer C2.2, C3.1, C4.2, C5.2
- net ADC SCL: now also R1.1
- net ADC SDA: now also R2.1
- net 8 - IRQ: now reaches U2.12 (P1.06)
- net 8 - IRQ: now also U1.8 (IRQ)
- net 4 - CSN: now reaches U2.15 (P1.11)
- net 4 - CSN: now also U1.4 (~{CSN})
- net 3 - CE: now reaches U2.33 (P1.07)
- net 3 - CE: now also U1.3 (CE)
- net sensor1 renamed out1
- net sensor2 renamed out2
- no-connect marks 3 -> 10
Other:
- moved on the sheet: D1, D2, D3, D4, R6, R7, R8, R9
