File: kicad smolslimes/deltavr trackers/deltavr trackers.kicad_pcb (KiCad board)
At the start: 2 copper layers, 1 part

Commit message: changes to deltavr smolslimes aka moth trackers
Parts:
- removed the REF** at (60.0, 65.0)
- added REF**: LGA14-L_2P59X3P1X0P5_STM, lsm6dsvtr footprint:LGA14-L_2P59X3P1X0P5_STM-M, F.Cu at (147.0, 102.5)
- added REF**: PinHeader_2x01_P1.00mm_Vertical, Connector_PinHeader_1.00mm:PinHeader_2x01_P1.00mm_Vertical, F.Cu at (150.0, 91.0)
- added U1: nice_nano, nicenano footprint:nice_nano, F.Cu at (126.0, 92.0)
